Commit message: WIP: Safety Ridgeback.

File: ridgeback_description/urdf/accessories.urdf.xacro (robot description, xacro)
@@ -35,3 +35,46 @@
                             location="-1" />
   </xacro:if>
+  <!-- If enabled, generate the front SICK S300 LASER payload.
+       This uses the same mesh as the lms1xx since they are the footprint
+       and the simulation parameters can be variable. -->
+  <xacro:if value="$(optenv RIDGEBACK_FRONT_S300_LASER 0)">
+    <xacro:sick_lms1xx_mount prefix="front"
+                            topic="front/scan"
+                            location="1" />
+  </xacro:if>
+  <!-- If enabled, generate the rear SICK S300 LASER payload. -->
+  <xacro:if value="$(optenv RIDGEBACK_REAR_S300_LASER 0)">
+    <xacro:sick_lms1xx_mount prefix="rear"
+                            topic="rear/scan"
+                            location="-1" />
+  </xacro:if>
+  <!-- If enabled, generate the optional Microstrain 3DM-GX2/3 IMU payload. -->
+  <xacro:if value="$(optenv RIDGEBACK_MICROSTRAIN_IMU 0)">
+    <link name="$(optenv RIDGEBACK_MICROSTRAIN_IMU_LINK upgraded)_imu_link" />
+    <joint name="$(optenv RIDGEBACK_MICROSTRAIN_IMU_MOUNT mid)_imu_joint" type="fixed">
+      <origin xyz="$(optenv RIDGEBACK_MICROSTRAIN_IMU_OFFSET 0 0 0)"
+              rpy="$(optenv RIDGEBACK_MICROSTRAIN_IMU_RPY 0 0 0)" />
+      <parent link="$(optenv RIDGEBACK_MICROSTRAIN_IMU_MOUNT mid)_mount" />
+      <child link="$(optenv RIDGEBACK_MICROSTRAIN_IMU_LINK upgraded)_imu_link" />
+    </joint>
+  </xacro:if>
+  <xacro:include filename="$(find pointgrey_camera_description)/urdf/pointgrey_flea3.urdf.xacro" />
+  <xacro:if value="$(optenv JACKAL_FLEA3 0)">
+    <camera_mount prefix="$(optenv JACKAL_FLEA3_MOUNT front)"
+                       tilt="$(optenv JACKAL_FLEA3_TILT 0.5236)"/>
+    <joint name="$(optenv JACKAL_FLEA3_MOUNT front)_camera_mount_joint" type="fixed">
+      <origin xyz="$(optenv JACKAL_FLEA3_OFFSET 0 0 0)"
+              rpy="$(optenv JACKAL_FLEA3_RPY 0 0 0)" />
+      <parent link="$(optenv JACKAL_FLEA3_MOUNT front)_mount" />
+      <child link="$(optenv JACKAL_FLEA3_MOUNT front)_camera_mount" />
+    </joint>
+    <pointgrey_flea3 frame="$(optenv JACKAL_FLEA3_MOUNT front)_camera" name="$(optenv JACKAL_FLEA3_NAME front)"
+      camera_x="0.0754" camera_y="0.029" camera_z="0.035"
+      camera_mass="0.085" hfov="1.0471975512" fps="60" width="640" height="512"/>
+    <joint name="$(optenv JACKAL_FLEA3_MOUNT front)_camera_bracket_joint" type="fixed">
+      <origin xyz="0.020 0 0.0245" rpy="0 0 0" />
+      <parent link="$(optenv JACKAL_FLEA3_MOUNT front)_camera_beam" />
+      <child link="$(optenv JACKAL_FLEA3_MOUNT front)_camera" />
+    </joint>
+  </xacro:if>
 </robot>

Commit message: [WIP] More changes.

File: ridgeback_description/urdf/accessories.urdf.xacro (robot description, xacro)
@@ -14,24 +14,24 @@
   <xacro:if value="$(optenv RIDGEBACK_FRONT_HOKUYO_LASER 0)">
     <xacro:hokuyo_ust-10lx_mount prefix="front"
-                            topic="front/scan"
-                            location="1" />
+                                 topic="front/scan"
+                                 location="1" />
   </xacro:if>
   <!-- If enabled, generate the rear HOKUYO UST-10LX LASER payload. -->
   <xacro:if value="$(optenv RIDGEBACK_REAR_HOKUYO_LASER 0)">
     <xacro:hokuyo_ust-10lx_mount prefix="rear"
-                            topic="rear/scan"
-                            location="-1" />
+                                 topic="rear/scan"
+                                 location="-1" />
   </xacro:if>
   <!-- If enabled, generate the front SICK LMS111 LASER payload. -->
   <xacro:if value="$(optenv RIDGEBACK_FRONT_SICK_LASER 0)">
     <xacro:sick_lms1xx_mount prefix="front"
-                            topic="front/scan"
-                            location="1" />
+                             topic="front/scan"
+                             location="1" />
   </xacro:if>
   <!-- If enabled, generate the rear SICK LMS111 LASER payload. -->
   <xacro:if value="$(optenv RIDGEBACK_REAR_SICK_LASER 0)">
     <xacro:sick_lms1xx_mount prefix="rear"
-                            topic="rear/scan"
-                            location="-1" />
+                             topic="rear/scan"
+                             location="-1" />
   </xacro:if>
   <!-- If enabled, generate the front SICK S300 LASER payload.
@@ -40,12 +40,12 @@
   <xacro:if value="$(optenv RIDGEBACK_FRONT_S300_LASER 0)">
     <xacro:sick_lms1xx_mount prefix="front"
-                            topic="front/scan"
-                            location="1" />
+                             topic="front/scan"
+                             location="1" />
   </xacro:if>
   <!-- If enabled, generate the rear SICK S300 LASER payload. -->
   <xacro:if value="$(optenv RIDGEBACK_REAR_S300_LASER 0)">
     <xacro:sick_lms1xx_mount prefix="rear"
-                            topic="rear/scan"
-                            location="-1" />
+                             topic="rear/scan"
+                             location="-1" />
   </xacro:if>
   <!-- If enabled, generate the optional Microstrain 3DM-GX2/3 IMU payload. -->
@@ -58,22 +58,36 @@
       <child link="$(optenv RIDGEBACK_MICROSTRAIN_IMU_LINK upgraded)_imu_link" />
     </joint>
+    <gazebo>
+      <plugin name="upgraded_imu_controller" filename="libhector_gazebo_ros_imu.so">
+        <robotNamespace>/</robotNamespace>
+        <updateRate>50.0</updateRate>
+        <bodyName>upgraded_imu_link</bodyName>
+        <topicName>upgraded_imu/data</topicName>
+        <accelDrift>0.005 0.005 0.005</accelDrift>
+        <accelGaussianNoise>0.005 0.005 0.005</accelGaussianNoise>
+        <rateDrift>0.005 0.005 0.005 </rateDrift>
+        <rateGaussianNoise>0.005 0.005 0.005 </rateGaussianNoise>
+        <headingDrift>0.005</headingDrift>
+        <headingGaussianNoise>0.005</headingGaussianNoise>
+      </plugin>
+    </gazebo>
   </xacro:if>
+  <!-- If enabled, generate the PointGrey Flea3 camera payload.. -->
   <xacro:include filename="$(find pointgrey_camera_description)/urdf/pointgrey_flea3.urdf.xacro" />
-  <xacro:if value="$(optenv JACKAL_FLEA3 0)">
-    <camera_mount prefix="$(optenv JACKAL_FLEA3_MOUNT front)"
-                       tilt="$(optenv JACKAL_FLEA3_TILT 0.5236)"/>
-    <joint name="$(optenv JACKAL_FLEA3_MOUNT front)_camera_mount_joint" type="fixed">
-      <origin xyz="$(optenv JACKAL_FLEA3_OFFSET 0 0 0)"
-              rpy="$(optenv JACKAL_FLEA3_RPY 0 0 0)" />
-      <parent link="$(optenv JACKAL_FLEA3_MOUNT front)_mount" />
-      <child link="$(optenv JACKAL_FLEA3_MOUNT front)_camera_mount" />
+  <xacro:if value="$(optenv RIDGEBACK_FLEA3 0)">
+    <joint name="$(optenv RIDGEBACK_FLEA3_MOUNT camera)_mount_joint" type="fixed">
+      <origin xyz="$(optenv RIDGEBACK_FLEA3_OFFSET 0 0 0)"
+              rpy="$(optenv RIDGEBACK_FLEA3_RPY 0 0 0)" />
+      <parent link="$(optenv RIDGEBACK_FLEA3_MOUNT mid)_mount" />
+      <child link="$(optenv RIDGEBACK_FLEA3_MOUNT camera)_mount" />
     </joint>
-    <pointgrey_flea3 frame="$(optenv JACKAL_FLEA3_MOUNT front)_camera" name="$(optenv JACKAL_FLEA3_NAME front)"
+   <link name="$(optenv RIDGEBACK_FLEA3_MOUNT camera)_mount" />
+    <pointgrey_flea3 frame="$(optenv RIDGEBACK_FLEA3_MOUNT camera)_link" name="$(optenv RIDGEBACK_FLEA3_NAME camera)"
       camera_x="0.0754" camera_y="0.029" camera_z="0.035"
       camera_mass="0.085" hfov="1.0471975512" fps="60" width="640" height="512"/>
-    <joint name="$(optenv JACKAL_FLEA3_MOUNT front)_camera_bracket_joint" type="fixed">
+    <joint name="$(optenv RIDGEBACK_FLEA3_MOUNT camera)_bracket_joint" type="fixed">
       <origin xyz="0.020 0 0.0245" rpy="0 0 0" />
-      <parent link="$(optenv JACKAL_FLEA3_MOUNT front)_camera_beam" />
-      <child link="$(optenv JACKAL_FLEA3_MOUNT front)_camera" />
+      <parent link="$(optenv RIDGEBACK_FLEA3_MOUNT camera)_mount" />
+      <child link="$(optenv RIDGEBACK_FLEA3_MOUNT camera)_link" />
     </joint>
   </xacro:if>

Commit message: [WIP] Material properties.

File: ridgeback_description/urdf/accessories.urdf.xacro (robot description, xacro)
@@ -58,18 +58,4 @@
       <child link="$(optenv RIDGEBACK_MICROSTRAIN_IMU_LINK upgraded)_imu_link" />
     </joint>
-    <gazebo>
-      <plugin name="upgraded_imu_controller" filename="libhector_gazebo_ros_imu.so">
-        <robotNamespace>/</robotNamespace>
-        <updateRate>50.0</updateRate>
-        <bodyName>upgraded_imu_link</bodyName>
-        <topicName>upgraded_imu/data</topicName>
-        <accelDrift>0.005 0.005 0.005</accelDrift>
-        <accelGaussianNoise>0.005 0.005 0.005</accelGaussianNoise>
-        <rateDrift>0.005 0.005 0.005 </rateDrift>
-        <rateGaussianNoise>0.005 0.005 0.005 </rateGaussianNoise>
-        <headingDrift>0.005</headingDrift>
-        <headingGaussianNoise>0.005</headingGaussianNoise>
-      </plugin>
-    </gazebo>
   </xacro:if>
   <!-- If enabled, generate the PointGrey Flea3 camera payload.. -->

File: ridgeback_description/urdf/accessories/hokuyo_ust-10lx_mount.urdf.xacro (robot description, xacro)
@@ -31,5 +31,5 @@
     </link>
     <gazebo reference="${prefix}_laser">
-      <turnGravityOff>true</turnGravityOff>
+      <turnGravityOff>false</turnGravityOff>
       <sensor type="ray" name="${prefix}_laser">
         <pose>0 0 0 0 0 0</pose>

File: ridgeback_description/urdf/accessories/microstrain_imu.urdf.xacro (robot description, xacro)
@@ -31,5 +31,5 @@
     </link>
     <gazebo reference="${prefix}_laser">
-      <turnGravityOff>true</turnGravityOff>
+      <turnGravityOff>false/turnGravityOff>
       <sensor type="ray" name="${prefix}_laser">
         <pose>0 0 0 0 0 0</pose>

File: ridgeback_description/urdf/ridgeback.urdf.xacro (robot description, xacro)
@@ -36,9 +36,9 @@
       <inertial>
         <origin xyz="0 0 0" rpy="0 0 0"/>
-        <mass value="0.477"/>
+        <mass value="2.3"/>
         <inertia
-          ixx="0.0013" ixy="0" ixz="0"
-          iyy="0.0024" iyz="0"
-          izz="0.0013"/>
+          ixx="3.3212e-3" ixy="0" ixz="0"
+          iyy="6.6424e-3" iyz="0"
+          izz="3.3212e-3"/>
       </inertial>
     </link>
@@ -70,9 +70,9 @@
       <inertial>
         <origin xyz="0 0 0" rpy="0 0 0"/>
-        <mass value="3"/>
+        <mass value="10.267"/>
         <inertia
-          ixx="0.001" ixy="0" ixz="0"
-          iyy="0.001" iyz="0"
-          izz="0.001"/>
+          ixx="0.0288" ixy="2.20484e-6" ixz="-1.3145e-5"
+          iyy="0.4324" iyz="1.8944e-3"
+          izz="0.4130"/>
       </inertial>
     </link>
@@ -112,16 +112,16 @@
     </visual>
     <collision>
-      <origin xyz="0 0 ${chassis_height/2}"/>
-      <geometry>
-        <box size="${chassis_length} ${chassis_width} ${chassis_height}"/>
+      <origin xyz="0 0 ${deck_height/2}"/>
+      <geometry>
+        <box size="${chassis_length} ${chassis_width} ${deck_height}"/>
       </geometry>
     </collision>
     <inertial>
       <origin xyz="0.012 0.002 0.067" rpy="0 0 0"/>
-      <mass value="50"/>
+      <mass value="165.304"/>
       <inertia
-        ixx="1.3136" ixy="0.0" ixz="0.0"
-        iyy="1.3922" iyz="0.0"
-        izz="2.0"/>
+        ixx="4.4744" ixy="0.03098" ixz="0.003647"
+        iyy="7.1624" iyz="0.1228"
+        izz="4.6155"/>
     </inertial>
   </link>
