Commit message: WIP: Added surface friction and fixed rocker inertia.

File: ridgeback_description/urdf/ridgeback.urdf.xacro (robot description, xacro)
@@ -69,5 +69,5 @@
       </visual>
       <inertial>
-        <origin xyz="0 0 0" rpy="0 0 0"/>
+        <origin xyz="0 0 0" rpy="${PI/2} 0 ${PI/2}"/>
         <mass value="10.267"/>
         <inertia
